Commit message: fine tune the locations of the camera, robot, and objects; replace some absolute paths with relative paths

File: src/ur_simulation_gz/ur_simulation_gz/urdf/camera_rgbd.urdf (robot description, URDF)
Before this commit: robot camera_rgbd, 2 links, 1 joints
Joints:
- joint camera_fixer_joint: origin xyz=0 0 0 rpy=0 1.57 -1.57 -> xyz=0 0 0 rpy=-1.57 1.57 -1.57

File: src/ur_simulation_gz/ur_simulation_gz/urdf/ur_gz.urdf.xacro (robot description, xacro)
@@ -59,5 +59,5 @@
     force_abs_paths="true"
     >
-    <origin xyz="0 0 0" rpy="0 0 0" />          <!-- position robot in the world -->
+    <origin xyz="0 0 0.7" rpy="0 0 0" />          <!-- position robot in the world -->
   </xacro:ur_robot>
   <gazebo reference="world">
